Commit message: Adjusting vnc screen size, putting in paths for materials

File: src/start_creating_robots/worlds_and_models/krytn/realsense_d435.urdf.xacro (robot description, xacro)
@@ -17,4 +17,5 @@
         </mesh>
       </geometry>
+      <origin xyz="0 0 0" rpy="0 0 ${pi/2}"/>
     </visual>
   </link>
